Commit message: Add xacro support with minimal geometry option for visualization
- Convert URDF to xacro with use_full_visual argument (default: false)
- Add minimal geometry GLB meshes for faster RViz rendering
- Update launch files to support use_full_visual parameter
- Remove unused OmniWheel.dae and old static URDF
- Default to minimal geometry, use_full_visual:=true for detailed meshes

Signed-off-by: Benjamin Perseghetti <bperseghetti@rudislabs.com>

File: spinali_optical_flow_description/urdf/spinali_optical_flow.urdf.xacro (robot description, xacro)
@@ -1,4 +1,12 @@
 <?xml version="1.0"?>
 <robot name="spinali_optical_flow" xmlns:xacro="http://ros.org/wiki/xacro">
+  <xacro:arg name="use_full_visual" default="false"/>
+  <xacro:property name="use_full_visual" value="$(arg use_full_visual)"/>
+  <!-- Z offset for minimal geometry meshes -->
+  <xacro:property name="minimal_z_offset" value="-0.0008"/>
+  <!-- Dark PCB green color for simple geometry -->
+  <material name="pcb_green">
+    <color rgba="0.0 0.3 0.15 1.0"/>
+  </material>
   <!-- World frame (fixed reference) -->
   <link name="world"/>
@@ -6,27 +14,45 @@
   <link name="spinali_optical_flow_link">
     <visual name="mcxn_t1_ofl">
-      <origin xyz="0 0 0" rpy="0 3.14159265358979323846 1.570796332769"/>
-      <geometry>
-        <mesh filename="package://spinali_optical_flow_description/meshes/OpticalFlow.glb" scale=".0254 .0254 .0254" />
-      </geometry>
+      <xacro:if value="${use_full_visual}">
+        <origin xyz="0 0 0" rpy="0 ${pi} ${pi/2}"/>
+        <geometry>
+          <mesh filename="package://spinali_optical_flow_description/meshes/OpticalFlow.glb" scale=".0254 .0254 .0254" />
+        </geometry>
+      </xacro:if>
+      <xacro:unless value="${use_full_visual}">
+        <origin xyz="0 0 ${minimal_z_offset}" rpy="${pi/2} 0 ${pi/2}"/>
+        <geometry>
+          <mesh filename="package://spinali_optical_flow_description/meshes/OpticalFlowMinimal.glb" scale="1 1 1" />
+        </geometry>
+      </xacro:unless>
     </visual>
     <visual name="mcxn_t1_hub">
-      <origin xyz="0 0 -0.00875" rpy="0 3.14159265358979323846 1.570796332769"/>
-      <geometry>
-        <mesh filename="package://spinali_optical_flow_description/meshes/MCXN947T1HubV0.glb" scale=".0254 .0254 .0254" />
-      </geometry>
+      <xacro:if value="${use_full_visual}">
+        <origin xyz="0 0 -0.00875" rpy="0 ${pi} ${pi/2}"/>
+        <geometry>
+          <mesh filename="package://spinali_optical_flow_description/meshes/MCXN947T1HubV0.glb" scale=".0254 .0254 .0254" />
+        </geometry>
+      </xacro:if>
+      <xacro:unless value="${use_full_visual}">
+        <origin xyz="0 0 ${-0.00865 + minimal_z_offset}" rpy="${pi/2} 0 ${pi/2}"/>
+        <geometry>
+          <mesh filename="package://spinali_optical_flow_description/meshes/MCXN947T1HubV0Minimal.glb" scale="1 1 1" />
+        </geometry>
+      </xacro:unless>
     </visual>
     <visual name="mcxn_t1_spacer">
-      <origin xyz="0.020 -0.01525 -0.0008" rpy="0 3.14159265358979323846 0"/>
+      <origin xyz="0.020 -0.01525 -0.0008" rpy="0 ${pi} 0"/>
       <geometry>
         <mesh filename="package://spinali_optical_flow_description/meshes/Spacer.glb" scale="1 1 1" />
       </geometry>
     </visual>
-    <!-- <visual name="mcxn_t1_base">
-      <origin xyz="0 0 -0.0135" rpy="0 3.14159265358979323846 -1.570796332769"/>
-      <geometry>
-        <mesh filename="package://spinali_optical_flow_description/meshes/Base.glb" scale="1 1 1" />
-      </geometry>
-    </visual> -->
+    <xacro:unless value="${use_full_visual}">
+      <visual name="mcxn_t1_base">
+        <origin xyz="0 0 -0.014" rpy="0 ${pi} ${-pi/2}"/>
+        <geometry>
+          <mesh filename="package://spinali_optical_flow_description/meshes/Base.glb" scale="1 1 1" />
+        </geometry>
+      </visual>
+    </xacro:unless>
   </link>
   <link name="afbr-s50lx85d"/>

Commit message: Add no_case option to exclude base and spacer from visualization
- Add no_case xacro argument (default: true) to exclude case components
- Update launch files to pass no_case parameter
- When no_case:=true, base and spacer meshes are not included
- Use no_case:=false to show the full enclosure

Signed-off-by: Benjamin Perseghetti <bperseghetti@rudislabs.com>

File: spinali_optical_flow_description/urdf/spinali_optical_flow.urdf.xacro (robot description, xacro)
@@ -3,4 +3,6 @@
   <xacro:arg name="use_full_visual" default="false"/>
   <xacro:property name="use_full_visual" value="$(arg use_full_visual)"/>
+  <xacro:arg name="no_case" default="true"/>
+  <xacro:property name="no_case" value="$(arg no_case)"/>
   <!-- Z offset for minimal geometry meshes -->
   <xacro:property name="minimal_z_offset" value="-0.0008"/>
@@ -41,17 +43,19 @@
       </xacro:unless>
     </visual>
-    <visual name="mcxn_t1_spacer">
-      <origin xyz="0.020 -0.01525 -0.0008" rpy="0 ${pi} 0"/>
-      <geometry>
-        <mesh filename="package://spinali_optical_flow_description/meshes/Spacer.glb" scale="1 1 1" />
-      </geometry>
-    </visual>
-    <xacro:unless value="${use_full_visual}">
-      <visual name="mcxn_t1_base">
-        <origin xyz="0 0 -0.014" rpy="0 ${pi} ${-pi/2}"/>
+    <xacro:unless value="${no_case}">
+      <visual name="mcxn_t1_spacer">
+        <origin xyz="0.020 -0.01525 -0.0008" rpy="0 ${pi} 0"/>
         <geometry>
-          <mesh filename="package://spinali_optical_flow_description/meshes/Base.glb" scale="1 1 1" />
+          <mesh filename="package://spinali_optical_flow_description/meshes/Spacer.glb" scale="1 1 1" />
         </geometry>
       </visual>
+      <xacro:unless value="${use_full_visual}">
+        <visual name="mcxn_t1_base">
+          <origin xyz="0 0 -0.014" rpy="0 ${pi} ${-pi/2}"/>
+          <geometry>
+            <mesh filename="package://spinali_optical_flow_description/meshes/Base.glb" scale="1 1 1" />
+          </geometry>
+        </visual>
+      </xacro:unless>
     </xacro:unless>
   </link>
